File: arisutea-pcb.kicad_pcb (KiCad board)
At the start: 2 copper layers, 339.1 x 121 mm, 177 parts, among them J10 PF6, J11 PF7, J12 VCC, J13 D+, J14 D-, J15 GND, J2 MISO, J3 VCC, J4 SCK, J5 MOSI, J6 RES, J7 GND, J8 PF4, J9 PF5, SW1 SW_Push, SW10 SW_Push, SW11 SW_Push, SW12 SW_Push, SW13 SW_Push, SW14 SW_Push, SW15 SW_Push, SW16 SW_Push, SW17 SW_Push, SW18 SW_Push, SW19 SW_Push, SW2 SW_Push, SW20 SW_Push, SW21 SW_Push, SW22 SW_Push, SW23 SW_Push, SW24 SW_Push, SW25 SW_Push, SW26 SW_Push, SW27 SW_Push, SW28 SW_Push, SW29 SW_Push, SW3 SW_Push, SW30 SW_Push, SW31 SW_Push, SW32 SW_Push, SW33 SW_Push, SW34 SW_Push, SW35 SW_Push, SW36 SW_Push, SW37 SW_Push, SW38 SW_Push, SW39 SW_Push, SW4 SW_Push, SW40 SW_Push, SW41 SW_Push, SW42 SW_Push, SW43 SW_Push, SW44 SW_Push, SW45 SW_Push, SW46 SW_Push, SW47 SW_Push, SW48 SW_Push, SW49 SW_Push, SW5 SW_Push, SW50 SW_Push, SW51 SW_Push, SW52 SW_Push, SW53 SW_Push, SW54 SW_Push, SW55 SW_Push, SW56 SW_Push, SW57 SW_Push, SW58 SW_Push, SW59 SW_Push, SW6 SW_Push, SW60 SW_Push, SW61 SW_Push, SW62 SW_Push, SW63 SW_Push, SW64 SW_Push, SW65 SW_Push, SW66 SW_Push, SW7 SW_Push, SW8 SW_Push, SW9 SW_Push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

Commit message: update switch positions to be more uniform
Parts:
- moved SW40 0.18 mm to (230.1, 83.7)
- moved SW36 0.16 mm to (220.1, 105.3)
- moved SW41 0.15 mm to (238.7, 101.4)
- moved SW48 0.15 mm to (258.8, 58.1)
- moved SW42 0.14 mm to (226.9, 45.5)
- moved SW51 0.13 mm to (265.6, 37.2)
- moved SW26 0.12 mm to (148.9, 89.6)
- moved SW38 0.12 mm to (208.3, 49.4)
- moved SW39 0.12 mm to (221.6, 66.0)
- moved SW45 0.12 mm to (257.3, 97.4)
- moved SW24 0.11 mm to (142.8, 49.3)
- moved SW32 0.11 mm to (201.4, 109.3)
- moved SW18 0.11 mm to (116.9, 102.3)
- moved SW19 0.11 mm to (124.2, 45.4)
- moved SW23 0.10 mm to (131.7, 124.9)
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Changed lines of the file:
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@@
     (40 Dwgs.User user)
     (41 Cmts.User user)
-    (42 Eco1.User user)
+    (42 Eco1.User user hide)
     (43 Eco2.User user hide)
     (44 Edge.Cuts user)
@@
   )
   (module arisutea:SW_Hotswap_Kailh_1.50u (layer F.Cu)
-    (at 322.199 57.785)
+    (at 322.136878 57.776625)
     (descr "Kailh keyswitch Hotswap Socket, ")
     (tags "Kailh Keyboard Keyswitch Switch Hotswap Socket 1.50u")
@@
   )
   (module arisutea:SW_Hotswap_Kailh_1.00u (layer F.Cu)
-    (at 265.557 37.338)
+    (at 265.583272 37.208803)
     (descr "Kailh keyswitch Hotswap Socket, ")
     (tags "Kailh Keyboard Keyswitch Switch Hotswap Socket 1.00u")
@@
   )
   (module arisutea:SW_Hotswap_Kailh_1.00u (layer F.Cu)
-    (at 258.699 58.166 12)
+    (at 258.84076 58.115293 12)
     (descr "Kailh keyswitch Hotswap Socket, ")
     (tags "Kailh Keyboard Keyswitch Switch Hotswap Socket 1.00u")
@@
   )
   (module arisutea:SW_Hotswap_Kailh_1.00u (layer F.Cu)
-    (at 245.491 41.402 12)
+    (at 245.478556 41.485038 12)
     (descr "Kailh keyswitch Hotswap Socket, ")
     (tags "Kailh Keyboard Keyswitch Switch Hotswap Socket 1.00u")
@@
   )
   (module arisutea:SW_Hotswap_Kailh_1.00u (layer F.Cu)
-    (at 251.968 117.983 12)
+    (at 251.975669 118.052781 12)
     (descr "Kailh keyswitch Hotswap Socket, ")
     (tags "Kailh Keyboard Keyswitch Switch Hotswap Socket 1.00u")
@@
   )
   (module arisutea:SW_Hotswap_Kailh_1.00u (layer F.Cu)
-    (at 257.302 97.282 12)
+    (at 257.340863 97.393743 12)
     (descr "Kailh keyswitch Hotswap Socket, ")
     (tags "Kailh Keyboard Keyswitch Switch Hotswap Socket 1.00u")
@@
   )
   (module arisutea:SW_Hotswap_Kailh_1.00u (layer F.Cu)
-    (at 240.157 62.103 12)
+    (at 240.212936 62.092765 12)
     (descr "Kailh keyswitch Hotswap Socket, ")
     (tags "Kailh Keyboard Keyswitch Switch Hotswap Socket 1.00u")
@@
   )
   (module arisutea:SW_Hotswap_Kailh_1.00u (layer F.Cu)
-    (at 226.949 45.339 12)
+    (at 226.879102 45.456229 12)
     (descr "Kailh keyswitch Hotswap Socket, ")
     (tags "Kailh Keyboard Keyswitch Switch Hotswap Socket 1.00u")
@@
   )
   (module arisutea:SW_Hotswap_Kailh_1.00u (layer F.Cu)
-    (at 238.76 101.219 12)
+    (at 238.718785 101.365066 12)
     (descr "Kailh keyswitch Hotswap Socket, ")
     (tags "Kailh Keyboard Keyswitch Switch Hotswap Socket 1.00u")
@@
   )
   (module arisutea:SW_Hotswap_Kailh_1.00u (layer F.Cu)
-    (at 230.251 83.566 12)
+    (at 230.135444 83.701372 12)
     (descr "Kailh keyswitch Hotswap Socket, ")
     (tags "Kailh Keyboard Keyswitch Switch Hotswap Socket 1.00u")
@@
   )
   (module arisutea:SW_Hotswap_Kailh_1.00u (layer F.Cu)
-    (at 221.615 65.913 12)
+    (at 221.587033 66.029659 12)
     (descr "Kailh keyswitch Hotswap Socket, ")
     (tags "Kailh Keyboard Keyswitch Switch Hotswap Socket 1.00u")
@@
   )
   (module arisutea:SW_Hotswap_Kailh_1.00u (layer F.Cu)
-    (at 208.153 49.403 12)
+    (at 208.273375 49.411604 12)
     (descr "Kailh keyswitch Hotswap Socket, ")
     (tags "Kailh Keyboard Keyswitch Switch Hotswap Socket 1.00u")
@@
   )
   (module arisutea:SW_Hotswap_Kailh_2.75u_RevStab (layer F.Cu)
-    (at 212.471 126.365 12)
+    (at 212.54567 126.405471 12)
     (descr "Kailh keyswitch Hotswap Socket, ")
     (tags "Kailh Keyboard Keyswitch Switch Hotswap Socket 2.75u")
@@
   )
   (module arisutea:SW_Hotswap_Kailh_1.00u (layer F.Cu)
-    (at 220.218 105.283 12)
+    (at 220.063535 105.305001 12)
     (descr "Kailh keyswitch Hotswap Socket, ")
     (tags "Kailh Keyboard Keyswitch Switch Hotswap Socket 1.00u")
@@
   )
   (module arisutea:SW_Hotswap_Kailh_1.00u (layer F.Cu)
-    (at 211.582 87.63 12)
+    (at 211.520878 87.647023 12)
     (descr "Kailh keyswitch Hotswap Socket, ")
     (tags "Kailh Keyboard Keyswitch Switch Hotswap Socket 1.00u")
@@
   )
   (module arisutea:SW_Hotswap_Kailh_1.00u (layer F.Cu)
-    (at 202.946 69.977 12)
+    (at 202.963458 70.013277 12)
     (descr "Kailh keyswitch Hotswap Socket, ")
     (tags "Kailh Keyboard Keyswitch Switch Hotswap Socket 1.00u")
@@
   )
   (module arisutea:SW_Hotswap_Kailh_1.00u (layer F.Cu)
-    (at 189.611 53.34 12)
+    (at 189.645551 53.366978 12)
     (descr "Kailh keyswitch Hotswap Socket, ")
     (tags "Kailh Keyboard Keyswitch Switch Hotswap Socket 1.00u")
@@
   )
   (module arisutea:SW_Hotswap_Kailh_1.00u (layer F.Cu)
-    (at 201.549 109.22 12)
+    (at 201.441212 109.255783 12)
     (descr "Kailh keyswitch Hotswap Socket, ")
     (tags "Kailh Keyboard Keyswitch Switch Hotswap Socket 1.00u")
@@
   )
   (module arisutea:SW_Hotswap_Kailh_1.00u (layer F.Cu)
-    (at 192.913 91.567 12)
+    (at 192.876017 91.618637 12)
     (descr "Kailh keyswitch Hotswap Socket, ")
     (tags "Kailh Keyboard Keyswitch Switch Hotswap Socket 1.00u")
@@
   )
   (module arisutea:SW_Hotswap_Kailh_1.00u (layer F.Cu)
-    (at 184.277 73.914 12)
+    (at 184.308862 73.98107 12)
     (descr "Kailh keyswitch Hotswap Socket, ")
     (tags "Kailh Keyboard Keyswitch Switch Hotswap Socket 1.00u")
@@
   )
   (module arisutea:SW_Hotswap_Kailh_1.00u (layer F.Cu)
-    (at 161.417 53.34 348)
+    (at 161.462926 53.264632 348)
     (descr "Kailh keyswitch Hotswap Socket, ")
     (tags "Kailh Keyboard Keyswitch Switch Hotswap Socket 1.00u")
@@
   )
   (module arisutea:SW_Hotswap_Kailh_1.00u (layer F.Cu)
-    (at 159.639 130.81 348)
+    (at 159.630614 130.831569 348)
     (descr "Kailh keyswitch Hotswap Socket, ")
     (tags "Kailh Keyboard Keyswitch Switch Hotswap Socket 1.00u")
@@
   )
   (module arisutea:SW_Hotswap_Kailh_1.00u (layer F.Cu)
-    (at 154.178 110.236 348)
+    (at 154.185801 110.17883 348)
     (descr "Kailh keyswitch Hotswap Socket, ")
     (tags "Kailh Keyboard Keyswitch Switch Hotswap Socket 1.00u")
@@
   )
   (module arisutea:SW_Hotswap_Kailh_1.00u (layer F.Cu)
-    (at 148.844 89.535 348)
+    (at 148.92566 89.624161 348)
     (descr "Kailh keyswitch Hotswap Socket, ")
     (tags "Kailh Keyboard Keyswitch Switch Hotswap Socket 1.00u")
@@
   )
   (module arisutea:SW_Hotswap_Kailh_1.00u (layer F.Cu)
-    (at 148.209 69.977 348)
+    (at 148.180612 69.954886 348)
     (descr "Kailh keyswitch Hotswap Socket, ")
     (tags "Kailh Keyboard Keyswitch Switch Hotswap Socket 1.00u")
@@
   )
   (module arisutea:SW_Hotswap_Kailh_1.00u (layer F.Cu)
-    (at 142.748 49.403 348)
+    (at 142.813005 49.309258 348)
     (descr "Kailh keyswitch Hotswap Socket, ")
     (tags "Kailh Keyboard Keyswitch Switch Hotswap Socket 1.00u")
@@
   )
   (module arisutea:SW_Hotswap_Kailh_2.00u_RevStab (layer F.Cu)
-    (at 131.572 124.841 348)
+    (at 131.655541 124.903964 348)
     (descr "Kailh keyswitch Hotswap Socket, ")
     (tags "Kailh Keyboard Keyswitch Switch Hotswap Socket 2.00u")
@@
   )
   (module arisutea:SW_Hotswap_Kailh_1.00u (layer F.Cu)
-    (at 135.509 106.299 348)
+    (at 135.517871 106.236035 348)
     (descr "Kailh keyswitch Hotswap Socket, ")
     (tags "Kailh Keyboard Keyswitch Switch Hotswap Socket 1.00u")
@@
   )
   (module arisutea:SW_Hotswap_Kailh_1.00u (layer F.Cu)
-    (at 130.302 85.598 348)
+    (at 130.280827 85.638153 348)
     (descr "Kailh keyswitch Hotswap Socket, ")
     (tags "Kailh Keyboard Keyswitch Switch Hotswap Socket 1.00u")
@@
   )
   (module arisutea:SW_Hotswap_Kailh_1.00u (layer F.Cu)
-    (at 129.54 66.04 348)
+    (at 129.535779 65.987504 348)
     (descr "Kailh keyswitch Hotswap Socket, ")
     (tags "Kailh Keyboard Keyswitch Switch Hotswap Socket 1.00u")
@@
   )
   (module arisutea:SW_Hotswap_Kailh_1.00u (layer F.Cu)
-    (at 124.206 45.466 348)
+    (at 124.191344 45.359934 348)
     (descr "Kailh keyswitch Hotswap Socket, ")
     (tags "Kailh Keyboard Keyswitch Switch Hotswap Socket 1.00u")
@@
   )
   (module arisutea:SW_Hotswap_Kailh_1.00u (layer F.Cu)
-    (at 116.967 102.235 348)
+    (at 116.876763 102.293239 348)
     (descr "Kailh keyswitch Hotswap Socket, ")
     (tags "Kailh Keyboard Keyswitch Switch Hotswap Socket 1.00u")
@@
   )
   (module arisutea:SW_Hotswap_Kailh_1.00u (layer F.Cu)
-    (at 111.633 81.661 348)
+    (at 111.635994 81.670771 348)
     (descr "Kailh keyswitch Hotswap Socket, ")
     (tags "Kailh Keyboard Keyswitch Switch Hotswap Socket 1.00u")
@@
   )
   (module arisutea:SW_Hotswap_Kailh_1.00u (layer F.Cu)
-    (at 110.871 61.976 348)
+    (at 110.889778 62.01517 348)
     (descr "Kailh keyswitch Hotswap Socket, ")
     (tags "Kailh Keyboard Keyswitch Switch Hotswap Socket 1.00u")
@@
   )
   (module arisutea:SW_Hotswap_Kailh_1.00u (layer F.Cu)
-    (at 99.06 117.983 348)
+    (at 99.013485 117.983956 348)
     (descr "Kailh keyswitch Hotswap Socket, ")
     (tags "Kailh Keyboard Keyswitch Switch Hotswap Socket 1.00u")
@@
   )
   (module arisutea:SW_Hotswap_Kailh_1.00u (layer F.Cu)
-    (at 98.298 98.298 348)
+    (at 98.262477 98.323622 348)
     (descr "Kailh keyswitch Hotswap Socket, ")
     (tags "Kailh Keyboard Keyswitch Switch Hotswap Socket 1.00u")
@@
   )
   (module arisutea:SW_Hotswap_Kailh_1.00u (layer F.Cu)
-    (at 92.964 77.724 348)
+    (at 92.991606 77.696916 348)
     (descr "Kailh keyswitch Hotswap Socket, ")
     (tags "Kailh Keyboard Keyswitch Switch Hotswap Socket 1.00u")

Commit message: library, silkscreen and gerber update
I moved all the footprints into a single library so that if folks don't have the particular lib they won't have to go and search for it or try to replace. Silkscreen was updated again to show clearer positioning of components and gerbers updated to most recent. Version number isn't changing as no big updates were made.
Parts:
- removed the LOGO1 at (286.3, 114.7)
- removed the LOGO1 at (289.1, 114.7)
- added LOGO1: arisutea_logo, arisutea:arisutea_logo, F.Cu at (287.8, 114.7)
- added LOGO2: arisutea_logo, arisutea:arisutea_logo, B.Cu at (287.4, 114.7)
- C1, C2, C3, C4, C5, C6, C7, C8, C9: footprint Capacitor_SMD:C_0805_2012Metric_Pad1.18x1.45mm_HandSolder -> arisutea:C_0805_2012Metric_Pad1.18x1.45mm_HandSolder
- D1, D10, D11, D12, D13, D14, D15, D16, D17, D18, D19, D2, D20, D21, D22, D23, D24, D25, D26, D27, D28, D29, D3, D30, D31, D32, D33, D34, D35, D36, D37, D38, D39, D4, D40, D41, D42, D43, D44, D45, D46, D47, D48, D49, D5, D50, D51, D52, D53, D54, D55, D56, D57, D58, D59, D6, D60, D61, D62, D63, D64, D65, D66, D7, D8, D9: footprint Diode_SMD:D_SOD-123 -> arisutea:D_SOD-123
- F1: footprint Fuse:Fuse_1206_3216Metric_Pad1.42x1.75mm_HandSolder -> arisutea:Fuse_1206_3216Metric_Pad1.42x1.75mm_HandSolder
- H1, H2, H3, H4, H5, H6, H7, H8: footprint Mounting_Keyboard_Stabilizer:THROUGH_HOLE_M2 -> arisutea:Plated_Through_Hole_M2
- J10, J11, J12, J13, J14, J15, J2, J3, J4, J5, J6, J7, J8, J9: footprint Connector_PinHeader_2.54mm:PinHeader_1x01_P2.54mm_Vertical -> arisutea:PinHeader_1x01_P2.54mm_Vertical
- R1, R2, R3, R4, R5, R6: footprint Resistor_SMD:R_0805_2012Metric_Pad1.20x1.40mm_HandSolder -> arisutea:R_0805_2012Metric_Pad1.20x1.40mm_HandSolder
- SWR1: footprint Button_Switch_SMD:SW_SPST_TL3342 -> arisutea:SW_SPST_TL3342
- U1: footprint Package_TO_SOT_SMD:SOT-23-6_Handsoldering -> arisutea:SOT-23-6_Handsoldering
- U2: footprint Package_QFP:TQFP-44_10x10mm_P0.8mm -> arisutea:TQFP-44_10x10mm_P0.8mm
- USB1: footprint USB_Type-C:USB_C_Receptacle_HRO_TYPE-C-31-M-12-HandSoldering -> arisutea:USB_C_Receptacle_HRO_TYPE-C-31-M-12-HandSoldering
- Y1: footprint Crystal:Crystal_SMD_TXC_7M-4Pin_3.2x2.5mm_HandSoldering -> arisutea:Crystal_SMD_TXC_7M-4Pin_3.2x2.5mm_HandSoldering
Routing:
- net /row0: track 322.8 -> 324.2 mm
- net /row1: track 388.1 -> 389.2 mm
- net /SCK: track 159.6 -> 160.3 mm
