File: arisutea-pcb.kicad_pcb (KiCad board)
At the start: 2 copper layers, 339.1 x 121 mm, 177 parts, among them J10 PF6, J11 PF7, J12 VCC, J13 D+, J14 D-, J15 GND, J2 MISO, J3 VCC, J4 SCK, J5 MOSI, J6 RES, J7 GND, J8 PF4, J9 PF5, SW1 SW_Push, SW10 SW_Push, SW11 SW_Push, SW12 SW_Push, SW13 SW_Push, SW14 SW_Push, SW15 SW_Push, SW16 SW_Push, SW17 SW_Push, SW18 SW_Push, SW19 SW_Push, SW2 SW_Push, SW20 SW_Push, SW21 SW_Push, SW22 SW_Push, SW23 SW_Push, SW24 SW_Push, SW25 SW_Push, SW26 SW_Push, SW27 SW_Push, SW28 SW_Push, SW29 SW_Push, SW3 SW_Push, SW30 SW_Push, SW31 SW_Push, SW32 SW_Push, SW33 SW_Push, SW34 SW_Push, SW35 SW_Push, SW36 SW_Push, SW37 SW_Push, SW38 SW_Push, SW39 SW_Push, SW4 SW_Push, SW40 SW_Push, SW41 SW_Push, SW42 SW_Push, SW43 SW_Push, SW44 SW_Push, SW45 SW_Push, SW46 SW_Push, SW47 SW_Push, SW48 SW_Push, SW49 SW_Push, SW5 SW_Push, SW50 SW_Push, SW51 SW_Push, SW52 SW_Push, SW53 SW_Push, SW54 SW_Push, SW55 SW_Push, SW56 SW_Push, SW57 SW_Push, SW58 SW_Push, SW59 SW_Push, SW6 SW_Push, SW60 SW_Push, SW61 SW_Push, SW62 SW_Push, SW63 SW_Push, SW64 SW_Push, SW65 SW_Push, SW66 SW_Push, SW7 SW_Push, SW8 SW_Push, SW9 SW_Push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

Commit message: 0.5 update
Fixes some routing that really did not need to be fixed but my OCD was screaming at me. Fixes an issue with the USB port only being shown as a through hole component and not an SMD. Reup gerbies, BOM and POS files.
Parts:
- J3: value VCC -> +5V
- J6: value RES -> ~RES~
- moved D54 2.69 mm to (297.9, 103.0)
- moved D50 2.69 mm to (271.7, 103.0)
- moved C9 1.15 mm to (189.2, 34.7)
- moved C3 0.76 mm to (184.8, 29.5)
- moved C4 0.76 mm to (182.5, 29.5)
- moved D10 0.13 mm to (78.4, 41.9)
- moved D29 0.11 mm to (153.7, 56.1)
- moved D11 0.11 mm to (84.0, 62.1)
- moved D60 0.10 mm to (315.1, 62.3)
- moved D56 0.10 mm to (291.2, 62.3)
- moved D1 0.06 mm to (40.3, 41.9)
Routing:
- net GND: track 77.8 -> 90.2 mm, vias 13 -> 18
- net +5V: track 173.9 -> 164.5 mm
- net /row4: track 437.9 -> 434.2 mm
- net Net-(D50-Pad2): track 5.32 -> 8.13 mm
- net Net-(D54-Pad2): track 5.32 -> 8.00 mm
- net /row3: track 444.6 -> 442.5 mm
- net /SCK: track 160.3 -> 158.2 mm
- net /PF4: track 35.9 -> 36.4 mm
- net /~RES~: track 41.0 -> 40.5 mm
Other:
- board text added: "Arisutea Rev 0.5 3x6 Designs mattyams"
- board text removed: "Arisutea Rev 0.4 3x6 Designs mattyams"

Commit message: added LED strip and indicator support, new cases for indicators
Parts:
- removed J10: PF6, arisutea:PinHeader_1x01_P2.54mm_Vertical
- removed J11: PF7, arisutea:PinHeader_1x01_P2.54mm_Vertical
- removed J8: PF4, arisutea:PinHeader_1x01_P2.54mm_Vertical
- removed J9: PF5, arisutea:PinHeader_1x01_P2.54mm_Vertical
- added J16: RGB, arisutea:PinHeader_1x03_P2.54mm_Vertical, B.Cu at (31.5, 52.6)
- added J17: RGB TO J18, arisutea:PinHeader_1x03_P2.54mm_Vertical, B.Cu at (339.2, 52.6)
- added J18: RGB FROM J17, arisutea:PinHeader_1x03_P2.54mm_Vertical, B.Cu at (355.0, 96.9)
- added LED1: NUM_LOCK, arisutea:LED_IN-S124ARUW, B.Cu at (138.7, 27.7)
- added LED2: CAPS_LOCK, arisutea:LED_IN-S124ARUW, B.Cu at (133.2, 27.7)
- added LED3: FN_LED, arisutea:LED_IN-S124ARUW, B.Cu at (127.8, 27.7)
- added R7: 470, arisutea:R_0805_2012Metric_Pad1.20x1.40mm_HandSolder, B.Cu at (141.2, 27.7)
- added R8: 470, arisutea:R_0805_2012Metric_Pad1.20x1.40mm_HandSolder, B.Cu at (135.8, 27.7)
- added R9: 470, arisutea:R_0805_2012Metric_Pad1.20x1.40mm_HandSolder, B.Cu at (130.3, 27.7)
- moved D32 0.19 mm to (195.4, 115.1)
- moved D36 0.15 mm to (214.1, 111.1)
- moved D48 0.13 mm to (252.3, 62.4)
- moved D25 0.11 mm to (140.4, 72.9)
- moved D41 0.10 mm to (232.8, 107.1)
- moved D47 0.07 mm to (239.4, 47.3)
Connections:
- U2 pad 36: /PF7 -> RGB
- U2 pad 37: /PF6 -> NUM_L
- U2 pad 38: /PF5 -> CAPS_L
- U2 pad 39: /PF4 -> FN_L
Routing:
- net GND: track 90.2 -> 677.1 mm, vias 18 -> 20
- net RGB: track 0.00 -> 170.4 mm, vias 0 -> 1
- net +5V: track 164.5 -> 312.4 mm
- net RGB_A: track 0.00 -> 50.8 mm
- net RGB_5V: track 0.00 -> 50.8 mm
- net NUM_L: track 0.00 -> 46.6 mm, vias 0 -> 2
- net /PF7: track 42.3 -> 0.00 mm, vias 1 -> 0
- net CAPS_L: track 0.00 -> 40.8 mm, vias 0 -> 2
- net /PF6: track 40.3 -> 0.00 mm, vias 1 -> 0
- net /PF5: track 38.4 -> 0.00 mm, vias 1 -> 0
- net /PF4: track 36.4 -> 0.00 mm, vias 1 -> 0
- net FN_L: track 0.00 -> 35.4 mm, vias 0 -> 2
- net Net-(LED3-PadA): track 0.00 -> 2.77 mm
- net Net-(LED2-PadA): track 0.00 -> 2.77 mm
- net Net-(LED1-PadA): track 0.00 -> 2.77 mm
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Other:
- board text added: "+5V"
- board text added: "Arisutea Rev 0.6 3x6 Design mattyams"
- board text added: "DATA"
- board text added: "Design Inspired by Fate Designs, CorruptedJef and robotictomato"
- board text added: "GND"
- board text removed: "Arisutea Rev 0.5 3x6 Designs mattyams"
- board text removed: "Original Design by Fate Designs, CorruptedJef and robotictomato"

Commit message: WS2812 PADS ADDED
Parts:
- removed J16: RGB, arisutea:PinHeader_1x03_P2.54mm_Vertical
- removed J17: RGB TO J18, arisutea:PinHeader_1x03_P2.54mm_Vertical
- removed J18: RGB FROM J17, arisutea:PinHeader_1x03_P2.54mm_Vertical
- added C10: 0.1uF, arisutea:C_0805_2012Metric_Pad1.18x1.45mm_HandSolder, B.Cu at (117.2, 28.3)
- added C11: 0.1uF, arisutea:C_0805_2012Metric_Pad1.18x1.45mm_HandSolder, B.Cu at (56.4, 27.4)
- added C12: 0.1uF, arisutea:C_0805_2012Metric_Pad1.18x1.45mm_HandSolder, B.Cu at (30.2, 46.7)
- added C13: 0.1uF, arisutea:C_0805_2012Metric_Pad1.18x1.45mm_HandSolder, B.Cu at (30.5, 88.1)
- added C14: 0.1uF, arisutea:C_0805_2012Metric_Pad1.18x1.45mm_HandSolder, B.Cu at (28.7, 124.1)
- added C15: 0.1uF, arisutea:C_0805_2012Metric_Pad1.18x1.45mm_HandSolder, B.Cu at (82.3, 126.3)
- added C16: 0.1uF, arisutea:C_0805_2012Metric_Pad1.18x1.45mm_HandSolder, B.Cu at (138.4, 133.5)
- added C17: 0.1uF, arisutea:C_0805_2012Metric_Pad1.18x1.45mm_HandSolder, B.Cu at (181.2, 139.4)
- added C18: 0.1uF, arisutea:C_0805_2012Metric_Pad1.18x1.45mm_HandSolder, B.Cu at (237.9, 128.1)
- added C19: 0.1uF, arisutea:C_0805_2012Metric_Pad1.18x1.45mm_HandSolder, B.Cu at (282.2, 124.8)
- added C20: 0.1uF, arisutea:C_0805_2012Metric_Pad1.18x1.45mm_HandSolder, B.Cu at (362.8, 125.5)
- added C21: 0.1uF, arisutea:C_0805_2012Metric_Pad1.18x1.45mm_HandSolder, B.Cu at (360.4, 88.1)
- added C22: 0.1uF, arisutea:C_0805_2012Metric_Pad1.18x1.45mm_HandSolder, B.Cu at (360.4, 29.1)
- added C23: 0.1uF, arisutea:C_0805_2012Metric_Pad1.18x1.45mm_HandSolder, B.Cu at (236.0, 28.3)
- added LED10: WS2812B, arisutea:LED_WS2812B, B.Cu at (132.8, 132.1)
- added LED11: WS2812B, arisutea:LED_WS2812B, B.Cu at (175.4, 139.3)
- added LED12: WS2812B, arisutea:LED_WS2812B, B.Cu at (232.3, 129.2)
- added LED13: WS2812B, arisutea:LED_WS2812B, B.Cu at (276.4, 124.8)
- added LED14: WS2812B, arisutea:LED_WS2812B, B.Cu at (358.1, 125.3)
- added LED15: WS2812B, arisutea:LED_WS2812B, B.Cu at (360.4, 93.9)
- added LED16: WS2812B, arisutea:LED_WS2812B, B.Cu at (360.4, 34.9)
- added LED17: WS2812B, arisutea:LED_WS2812B, B.Cu at (241.7, 28.3)
- added LED4: WS2812B, arisutea:LED_WS2812B, B.Cu at (112.0, 28.2)
- added LED5: WS2812B, arisutea:LED_WS2812B, B.Cu at (61.3, 27.7)
- added LED6: WS2812B, arisutea:LED_WS2812B, B.Cu at (30.1, 40.9)
- added LED7: WS2812B, arisutea:LED_WS2812B, B.Cu at (30.4, 82.0)
- added LED8: WS2812B, arisutea:LED_WS2812B, B.Cu at (28.7, 118.4)
- added LED9: WS2812B, arisutea:LED_WS2812B, B.Cu at (75.6, 124.2)
- added LOGO3: arisutea_logo, Symbol:OSHW-Logo_5.7x6mm_SilkScreen, B.Cu at (59.2, 111.5)
- added LOGO4: arisutea_logo, Symbol:OSHW-Logo_5.7x6mm_SilkScreen, F.Cu at (59.2, 111.5)
- added LOGO5: arisutea_logo, arisutea:QMK_Logo_Dark, F.Cu at (74.3, 111.8)
- added LOGO6: QMK_LOGO, arisutea:QMK_Logo_Dark, B.Cu at (74.3, 111.8)
- added R10: 720, arisutea:R_0805_2012Metric_Pad1.20x1.40mm_HandSolder, B.Cu at (115.7, 32.4)
- moved D28 1.26 mm to (151.9, 132.5)
- moved D23 1.01 mm to (124.0, 126.9)
Routing:
- net +5V: track 312.4 -> 974.3 mm
- net GND: track 677.1 -> 912.7 mm, vias 20 -> 29
- net Net-(LED16-Pad2): track 0.00 -> 123.3 mm
- net RGB: track 170.4 -> 58.1 mm, vias 1 -> 2
- net Net-(LED13-Pad2): track 0.00 -> 80.2 mm
- net Net-(LED15-Pad2): track 0.00 -> 58.0 mm
- net Net-(LED11-Pad2): track 0.00 -> 57.0 mm
- net Net-(LED10-Pad4): track 0.00 -> 55.8 mm
- net RGB_A: track 50.8 -> 0.00 mm
- net RGB_5V: track 50.8 -> 0.00 mm
- net Net-(LED8-Pad2): track 0.00 -> 50.0 mm
- net Net-(LED4-Pad2): track 0.00 -> 46.9 mm
- net Net-(LED12-Pad2): track 0.00 -> 41.8 mm
- net Net-(LED10-Pad2): track 0.00 -> 41.5 mm
- net Net-(LED6-Pad2): track 0.00 -> 38.5 mm
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